File: schematics/alte_designs/first.sch (EAGLE design)
At the start: 167 parts, among them IC1 4093D, IC2 AT-MEGA-8, IC4 ATMEGA2560-16AU, T1 Farnell: 1299313, T2 Farnell: 1299313, T3 Farnell: 1299313, T4 T-IRLMS6702, T5 Farnell: 1299313

Commit message: new input resistor layout, pull ups pull down, new diode, new connector for soldering
Parts:
- removed C8: 100nF, RCLDT:C0805
- removed D1, D2, D8, D9: 5.5V, diode:ZENER-DIODESOD80C
- removed D12: 20V, diode:ZENER-DIODESOD80C
- removed R42, R43, R44, R46, R47: n.b. / 0R, RCLDT:R0805
- removed R45, R48, R49, R_EXT13, R_EXT14, R_EXT15, R_EXT16: n.b., RCLDT:R0805
- removed R_DZ_DIV2: 3k3, RCLDT:R0805
- removed R_EXT10, R_EXT11, R_EXT7: 10k, RCLDT:R0805
- removed R_EXT12, R_EXT8, R_EXT9: 5k, RCLDT:R0805
- removed U$1: SPEEDOSTECKER, Kolja:SPEEDOSTECKER
- added D14, D15: SS24, RCLDT:D-SSMB-A+K
- added D45: SM6T30V, RCLDT:D-TD
- added JP10, JP11, JP12, JP13, JP14, JP15, JP16, JP17, JP18, JP19, JP20, JP3, JP4, JP5, JP6, JP7, JP8, JP9: (no value), pinhead:PINHD-1X1
- added R_EXT1, R_EXT2, R_EXT5, R_EXT6: n.b., RCLDT:R0805
- added R_EXT3, R_EXT4: 5k, RCLDT:R0805
- added S2: U, SWITCH+RELAIS:SW-TASTERECO-DIAGONAL
- added S3: R, SWITCH+RELAIS:SW-TASTERECO-DIAGONAL
- added S4: D, SWITCH+RELAIS:SW-TASTERECO-DIAGONAL
- added S5: L, SWITCH+RELAIS:SW-TASTERECO-DIAGONAL
- added TX2: (no value), pinhead:PINHD-1X2
- added X2: SUB-D-IP67, Kolja2:SUB-D-IP67
- D18, D19: value n.b. / 20V-ZD. -> 20V-ZD.; device diode:ZENER-DIODESOD80C -> diode:ZENER-DIODESMB
- D6: device diode:ZENER-DIODESOD80C -> diode:ZENER-DIODESMB
- R38: value n.b. -> 0R
- R7: value n.b. / 5k (Reed) -> 310R
- R8: value n.b. -> 310R
- R9: value n.b. / 0R -> 10k
Connections:
- removed net BL_L_IN: D2.C, IC4.(T3/INT6)PE6, R_EXT7.2, R_EXT8.1
- removed net BL_L_IN_H: R_EXT7.1, U$1.FLASH_L
- removed net BL_R_IN: D1.C, IC4.(CLKO/ICP3/INT7)PE7, R_EXT10.2, R_EXT9.1
- removed net BL_R_IN_H: R_EXT10.1, U$1.FLASH_R
- removed net HB_IN: D8.C, IC4.PH2(XCK2), R_EXT11.2, R_EXT12.1
- removed net HB_IN_H: R_EXT11.1, U$1.HIGH_BEAM
- removed net N$38 (its old number): IC1C.I1, R39.1, R44.2, R8.1, R9.2
- removed net N$41: D19.C, R46.1, U$1.EX_IN_OUT_D2
- removed net N$42: D18.C, R9.1, U$1.EX_IN_OUT_D1
- removed net N$43: R43.1, U$1.EX_IN_OUT_A2
- removed net N$44: R42.1, U$1.EX_IN_OUT_A1
- removed net N$45: IC1B.I1, R45.1, R46.2, R47.2, R49.1
- removed net N$46: IC1B.O, R48.1
- removed net NG_IN: IC4.PH1(TXD2), U$1.NEUTRAL_GEAR
- removed net OIL_PR_IN: IC4.PH0(RXD2), U$1.OIL_PRESSURE
- new net BL_L: R8.1, X2.8
- new net BL_R: R7.1, X2.7
- new net EXTEND1: D19.C, IC1B.I1, R_EXT4.2
- new net EXTEND2: D18.C, IC1C.I1, R_EXT3.2
- new net E_B_D: JP14.1, S4.2
- new net E_B_L: JP15.1, S5.2
- new net E_B_R: JP13.1, S3.2
- new net E_B_U: JP12.1, S2.2
- new net E_GND: JP16.1, JP17.1, JP18.1, JP19.1, JP20.1, S2.1, S3.1, S4.1, S5.1
- new net HIGH_BEAM: R6.1, X2.9
- new net N$11: D15.A, R4.1, R7.2
- new net N$2: D14.A, R1.1, R8.2
- new net N$78: R_EXT4.1, X2.14
- new net N$79: R39.1, R_EXT2.1, R_EXT3.1, X2.13
- new net N_IN: R27.1, X2.10
- new net OIL_PRESSURE: R5.1, X2.6
- new net RX2: IC4.PH0(RXD2)
- new net TX2: IC4.PH1(TXD2)
- net 12V: now also X2.11; no longer U$1.VIN
- net 12V_SAFE: now also D45.K; no longer D12.C
- net A0: now also R_EXT1.1, X2.15; no longer R42.2, R_EXT13.2, R_EXT15.1
- net A1: now also X2.5; no longer U$1.OIL_TEMP
- net A2: no longer D9.C
- net A7: now also R_EXT2.2, R_EXT5.1, R_EXT6.1; no longer R43.2, R_EXT14.2, R_EXT16.1
- net B_D: now also JP5.1
- net B_L: now also JP6.1
- net B_R: now also JP4.1
- net B_U: now also JP3.1
- net D42: now also TX2.1; no longer R6.1
- net D43: now also TX2.2; no longer R27.1
- net D44: no longer R1.1
- net D45: no longer R4.1
- net D46: no longer R5.1
- net D48: now also X2.12; no longer U$1.MC_COI
- net D49: now also IC1B.O; no longer R48.2, R49.2
- net D5: now also D14.K, D15.K, R9.2
- net DZ: no longer C8.1, R_DZ_DIV2.1
- net DZ_IN: now also X2.4; no longer U$1.DZ
- net GND: now also D45.A, JP10.1, JP11.1, JP7.1, JP8.1, JP9.1, R9.1, R_EXT6.2, X2.1; no longer C8.2, D1.A, D12.A, D2.A, D8.A, D9.A, R44.1, R47.1, R_DZ_DIV2.2, R_EXT12.2, R_EXT15.2, R_EXT16.2, R_EXT8.2, R_EXT9.2, U$1.GND
- net KUPPLUNG_IN: now also X2.2; no longer U$1.KUPPLUNG_IN
- net REED: no longer R7.2
- net REED_IN: now also X2.3; no longer U$1.REED
- net VDD: now also R_EXT1.2, R_EXT5.2; no longer R45.2, R7.1, R8.2, R_EXT13.1, R_EXT14.1
Other:
- note added: "Blinker"
- note added: "Ex_INOUT"
- note added: "Extension Header"
- note added: "Oil_in"
- note added: "Polarität checken!!"
- note removed: "1. Digitaler INOUT"
- note removed: "12V"
- note removed: "2. Digitaler IN via Schmidt"
- note removed: "3. Digitaler IN 12V"
- note removed: "?"
- note removed: "BL_L_OUT"
- note removed: "BL_R_OUT"
- note removed: "Connect"
- note removed: "Floatet das? Warum ist da kein Pullup?"
- note removed: "HB_OUT"
- note removed: "High Beam"
- note removed: "Left Flasher"
- note removed: "NG_OUT"
- note removed: "NOT(1&&2)"
- note removed: "NOT(12&&13)"
- note removed: "Neutral Gear"
- note removed: "OIL_PR_OUT"
- note removed: "Oil Preasure"
- note removed: "R ggn Masse"
- note removed: "Right Flasher"
- note removed: "Sw ggn M / Pulse?"
- note removed: "low active"
- note removed: "neu"
- moved on the sheet: 12V_F1, 5V_F, BAT_CLIP1, C11, C18, C38, C39, C4, C46, C49, C5, C6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
