File: schematics/alte_designs/v6/v6.brd (EAGLE design)
At the start: 159.4 x 94.4 mm, 174 parts, among them IC1 4093D, IC2 AT-MEGA-8, IC4 ATMEGA2560-16AU, T1 Farnell: 1299313, T2 Farnell: 1299313, T3 Farnell: 1299313, T4 T-IRLMS6702, T5 Farnell: 1299313

Commit message: Water compare resistor added
Parts:
- R_EXT1: value n.b. -> 390R
Changed lines of the file:
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@@
 <element name="R_SD_PWR_UP" library="resistor" package="M0805" value="10k" x="14.125" y="53.175"/>
 <element name="T5" library="RCLDT" package="SOT-23" value="Farnell: 1299313 " x="99.1" y="41.5" rot="MR270"/>
-<element name="R_EXT1" library="RCLDT" package="0805" value="n.b." x="27.8" y="38.5" rot="R270"/>
+<element name="R_EXT1" library="RCLDT" package="0805" value="390R" x="27.8" y="38.5" rot="R270"/>
 <element name="ST3" library="Stift+Buchsenleisten" package="BL17SMD_1X4" value="" x="67.7" y="43" rot="MR0">
 <attribute name="PACKAGE" value="SMD liegend L=7mm" x="67.7" y="43" size="1.778" layer="28" rot="MR0" display="off"/>
