File: schematics/alte_designs/v6/v6.sch (EAGLE design)
At the start: 174 parts, among them IC1 4093D, IC2 AT-MEGA-8, IC4 ATMEGA2560-16AU, T1 Farnell: 1299313, T2 Farnell: 1299313, T3 Farnell: 1299313, T4 T-IRLMS6702, T5 Farnell: 1299313, X2 SUB-D-IP67

Commit message: Water compare resistor added
Parts:
- R_EXT1: value n.b. -> 390R
Changed lines of the file:
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@@
 <part name="R_SD_PWR_UP" library="resistor" deviceset="R-EU_" device="M0805" value="10k"/>
 <part name="T5" library="RCLDT" deviceset="T-P-FET" device="BSS139" value="Farnell: 1299313 "/>
-<part name="R_EXT1" library="RCLDT" deviceset="R" device="0805" value="n.b."/>
+<part name="R_EXT1" library="RCLDT" deviceset="R" device="0805" value="390R"/>
 <part name="SUPPLY1" library="supply2" deviceset="VDD" device=""/>
 <part name="GND10" library="supply1" deviceset="GND" device=""/>
