File: schematics/plugins/canbus_shield-v1.brd (EAGLE design)
At the start: 31.5 x 43.4 mm, 17 parts, among them Q1 16MHz, U4 MCP2515, U5 MCP2551

Commit message: Fixed Airwire
Routing:
- net VCC: track 28.3 -> 35.6 mm
Changed lines of the file:
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@@
 <?xml version="1.0" encoding="utf-8"?>
 <!DOCTYPE eagle SYSTEM "eagle.dtd">
-<eagle version="6.2">
+<eagle version="6.4">
 <drawing>
 <settings>
@@
 </class>
 </classes>
-<designrules>
+<designrules name="default">
 <description language="de">&lt;b&gt;EAGLE Design Rules&lt;/b&gt;
 &lt;p&gt;
@@
 <wire x1="19.7" y1="20.4" x2="19.7" y2="18.95" width="0.254" layer="1"/>
 <wire x1="18.03" y1="37.83" x2="18.17" y2="37.74" width="0" layer="19" extent="1-1"/>
-<wire x1="23.865" y1="15.93" x2="19.7" y2="18.95" width="0" layer="19" extent="1-1"/>
+<wire x1="23.865" y1="15.93" x2="23.865" y2="18.335" width="0.254" layer="1"/>
+<wire x1="23.865" y1="18.335" x2="22.7" y2="19.5" width="0.254" layer="1"/>
+<wire x1="22.7" y1="19.5" x2="20.3" y2="19.5" width="0.254" layer="1"/>
+<wire x1="20.3" y1="19.5" x2="19.7" y2="18.9" width="0.254" layer="1"/>
+<wire x1="19.7" y1="18.9" x2="19.7" y2="18.95" width="0.254" layer="1"/>
 </signal>
 <signal name="MISO">
@@
 </signal>
 </signals>
-<errors>
-</errors>
 </board>
 </drawing>
