File: schematics/alte_designs/v7/JKW_standalone.brd (EAGLE design)
At the start: 159.4 x 80.7 mm, 241 parts, among them IC1 4093D, IC4 ATMEGA2560-16AU, Q1 BSS84, Q10 BSS84, Q11 BSS84, Q2 BSS84, Q3 BSS84, Q4 BSS84, Q5 BSS84, Q6 BSS84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

Commit message: Added low pass to reed signal, have to check the correct value (200nF?)
Parts:
- R_REED_DOWN: value 5k / n.b. (Reed / 5V Honda Signal) -> 5k (12V Honda Signal) / 100nF (Reed)
Changed lines of the file:
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@@
 <?xml version="1.0" encoding="utf-8"?>
 <!DOCTYPE eagle SYSTEM "eagle.dtd">
-<eagle version="6.2">
+<eagle version="6.4">
 <drawing>
 <settings>
@@
 </class>
 </classes>
-<designrules>
+<designrules name="default">
 <description language="de">DRC von Lutz
 Via´s bis 0.6mm mit Lötstoplack überzogen
@@
 <attribute name="NAME" x="133.1325" y="50.9975" size="0.6096" layer="26" rot="MR90"/>
 </element>
-<element name="R_REED_DOWN" library="RCLDT" package="0805" value="5k / n.b. (Reed / 5V Honda Signal)" x="38.6" y="17.525" smashed="yes" rot="R90">
+<element name="R_REED_DOWN" library="RCLDT" package="0805" value="5k (12V Honda Signal) / 100nF (Reed)" x="38.6" y="17.525" smashed="yes" rot="R90">
 <attribute name="NAME" x="38.5325" y="15.7275" size="0.6096" layer="25" rot="R270"/>
 </element>
