File: schematics/alte_designs/v7/JKW_standalone.sch (EAGLE design)
At the start: 241 parts, among them IC1 4093D, IC4 ATMEGA2560-16AU, Q1 BSS84, Q10 BSS84, Q11 BSS84, Q2 BSS84, Q3 BSS84, Q4 BSS84, Q5 BSS84, Q6 BSS84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

Commit message: Added low pass to reed signal, have to check the correct value (200nF?)
Parts:
- R_REED_DOWN: value 5k / n.b. (Reed / 5V Honda Signal) -> 5k (12V Honda Signal) / 100nF (Reed)
Changed lines of the file:
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@@
 <?xml version="1.0" encoding="utf-8"?>
 <!DOCTYPE eagle SYSTEM "eagle.dtd">
-<eagle version="6.2">
+<eagle version="6.4">
 <drawing>
 <settings>
@@
 <part name="R_OIL" library="RCLDT" deviceset="R" device="0805" value="52R"/>
 <part name="R_HIGHB" library="RCLDT" deviceset="R" device="0805" value="46R"/>
-<part name="R_REED_DOWN" library="RCLDT" deviceset="R" device="0805" value="5k / n.b. (Reed / 5V Honda Signal)"/>
+<part name="R_REED_DOWN" library="RCLDT" deviceset="R" device="0805" value="5k (12V Honda Signal) / 100nF (Reed)"/>
 <part name="U$12" library="SUPPLY" deviceset="GND" device=""/>
 <part name="R_REED" library="RCLDT" deviceset="R" device="0805" value="7k "/>
