File: schematics/SmartSpeedo/alte_designs/v1/SmartSpeedo.brd (EAGLE design)
At the start: 98.7 x 57.5 mm, 145 parts, among them IC1 4093D, IC2 L9637D, IC4 ATMEGA2560-16AU, T1 BC847, T13 Mouser: 771-2N7002BK215 , N-C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, T2 BC847, U4 MCP2515, U5 MCP2551

Commit message: Repaired Design (5V Diode)
Parts:
- removed D18: 78-MMBZ5232B-V, diode:SOT23
- added D15: 5.5V, diode:SOT23
- D6: value 20V-Zdiode -> 5.5V
Connections:
- net GND: now also D15.1; no longer D18.1
- net N$90: now also D15.3; no longer D18.3
Changed lines of the file:
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@@
 <?xml version="1.0" encoding="utf-8"?>
 <!DOCTYPE eagle SYSTEM "eagle.dtd">
-<eagle version="6.5.0">
+<eagle version="6.4">
 <drawing>
 <settings>
@@
 <attribute name="NAME" x="93.056" y="30.939" size="0.8128" layer="26" rot="MR90"/>
 </element>
-<element name="D6" library="diode" package="SOT23" value="20V-Zdiode" x="66.19" y="3.5" smashed="yes">
-<attribute name="NAME" x="62.484" y="3.393" size="0.6096" layer="26" rot="MR0"/>
-</element>
 <element name="S1" library="SWITCH+RELAIS" package="SW-ECO" value="" x="18.91" y="25.995" smashed="yes" rot="R90">
 <attribute name="NAME" x="19.475" y="22.2275" size="0.8128" layer="25" rot="R180"/>
@@
 <element name="D_VERPOL" library="RCLDT" package="SMB" value="SS24T3G" x="58.25" y="44.5" smashed="yes" rot="R90">
 <attribute name="NAME" x="60.9491" y="44.0118" size="0.6096" layer="25" rot="R90"/>
-</element>
-<element name="D18" library="diode" package="SOT23" value="78-MMBZ5232B-V" x="41.55" y="40.65" smashed="yes" rot="MR180">
-<attribute name="NAME" x="40.245" y="38.445" size="1.27" layer="26" rot="MR180"/>
-<attribute name="VALUE" x="39.645" y="43.825" size="1.27" layer="28" rot="MR180"/>
 </element>
 <element name="R_V_LOW" library="RCLDT" package="0805" value="1k" x="7.15" y="31.6" smashed="yes">
@@
 <element name="500MA_LITTLEFUSE" library="resistor" package="R1210" value="1210L050YR" x="95.8" y="45.5" rot="R270"/>
 <element name="700MA_LITTLEFUSE" library="resistor" package="R1210" value="1210L075YR" x="55.1" y="50.7"/>
+<element name="D6" library="diode" package="SOT23" value="5.5V" x="66.2" y="3.5"/>
+<element name="D15" library="diode" package="SOT23" value="5.5V" x="41.5" y="40.8" rot="MR180"/>
 </elements>
 <signals>
@@
 <contactref element="D5" pad="2"/>
 <contactref element="RX_L" pad="1"/>
-<contactref element="D6" pad="1"/>
 <contactref element="S1" pad="1"/>
 <contactref element="C11" pad="2"/>
 <contactref element="C18" pad="2"/>
 <contactref element="R_REED_DOWN" pad="2"/>
-<contactref element="D18" pad="1"/>
 <contactref element="R_V_LOW" pad="2"/>
 <contactref element="5V_SUPPLY" pad="GND"/>
@@
 <wire x1="21.26" y1="18.7" x2="21.26" y2="20.04" width="0.254" layer="16"/>
 <wire x1="21.26" y1="20.04" x2="21.1" y2="20.2" width="0.254" layer="16"/>
+<contactref element="D6" pad="1"/>
+<contactref element="D15" pad="1"/>
 </signal>
 <signal name="DZ">
 <contactref element="R_DZ" pad="2"/>
-<contactref element="D6" pad="3"/>
 <contactref element="IC1" pad="2"/>
 <contactref element="R_DZ_DOWN" pad="1"/>
@@
 <wire x1="70.6" y1="6.116" x2="69.3" y2="4.816" width="0.254" layer="1"/>
 <wire x1="62.708" y1="4.924" x2="62.8" y2="4.816" width="0.254" layer="1"/>
-<wire x1="69.3" y1="4.816" x2="66.106" y2="4.816" width="0.254" layer="1"/>
-<wire x1="66.106" y1="4.816" x2="66.19" y2="4.6" width="0.254" layer="1"/>
 <wire x1="60.3872" y1="4.824" x2="62.792" y2="4.824" width="0.254" layer="1"/>
 <wire x1="62.792" y1="4.824" x2="62.8" y2="4.816" width="0.254" layer="1"/>
-<wire x1="62.8" y1="4.816" x2="66.106" y2="4.816" width="0.254" layer="1"/>
+<wire x1="62.8" y1="4.816" x2="69.3" y2="4.816" width="0.254" layer="1"/>
+<contactref element="D6" pad="3"/>
+<wire x1="69.3" y1="4.816" x2="66.2" y2="4.6" width="0" layer="19" extent="1-1"/>
 </signal>
 <signal name="N$19">
@@
 </signal>
 <signal name="N$90">
-<contactref element="D18" pad="3"/>
 <contactref element="R_HB3" pad="2"/>
 <contactref element="R_E1_1" pad="1"/>
 <wire x1="41.6" y1="37.516" x2="41.55" y2="37.566" width="0.254" layer="16"/>
-<wire x1="41.55" y1="37.566" x2="41.55" y2="39.55" width="0.254" layer="16"/>
-<wire x1="41.55" y1="39.55" x2="41.716" y2="39.384" width="0.254" layer="16"/>
 <wire x1="41.716" y1="39.384" x2="45" y2="39.384" width="0.254" layer="16"/>
+<contactref element="D15" pad="3"/>
+<wire x1="41.5" y1="39.7" x2="41.6" y2="39.7" width="0.254" layer="16"/>
+<wire x1="41.6" y1="39.7" x2="41.6" y2="37.516" width="0.254" layer="16"/>
+<wire x1="41.6" y1="39.7" x2="41.716" y2="39.7" width="0.254" layer="16"/>
+<wire x1="41.716" y1="39.7" x2="41.716" y2="39.384" width="0.254" layer="16"/>
 </signal>
 <signal name="N$92">
@@
 </signal>
 </signals>
-<errors>
-</errors>
 </board>
 </drawing>
